Commit message: ignore .vscode. commit mara/ src folders

File: mara/mara_description/urdf/reinforcement_learning/mara_robot_gripper_140_camera_run.urdf.xacro (robot description, xacro)
@@ -91,5 +91,5 @@
   </joint>
   <joint name="camera_support2_to_camera" type="fixed">
-    <origin rpy="0 0 0" xyz="0 0.018 0.012"/>
+    <origin rpy="1.57 0 0" xyz="0 0.018 0.012"/>
     <parent link="camera_support2_link"/>
     <child link="camera_link"/>

File: mara/mara_description/urdf/reinforcement_learning/mara_robot_gripper_140_camera_train.urdf.xacro (robot description, xacro)
@@ -91,5 +91,5 @@
   </joint>
   <joint name="camera_support2_to_camera" type="fixed">
-    <origin rpy="0 0 0" xyz="0 0.018 0.012"/>
+    <origin rpy="1.57 0 0" xyz="0 0.018 0.012"/>
     <parent link="camera_support2_link"/>
     <child link="camera_link"/>
