Commit message: update camera setup on robot

File: mara/mara_description/urdf/reinforcement_learning/mara_robot_gripper_140_camera_train.urdf (robot description, URDF)
Before this commit: robot mara, 30 links, 29 joints
Joints:
- joint camera_support2_to_camera: origin xyz=0 0.018 0.012 rpy=0 0 0 -> xyz=0 0.018 0.012 rpy=1.57 0 0
